Commit message: commented out the advertise on the add gorup service. works for x_demo gazebo.

File: hebiros_description/urdf/myArm.urdf (robot description, URDF)
Before this commit: robot CNU_HEBI_Arm, 11 links, 10 joints
Links:
- removed link HEBI/base/INPUT_INTERFACE
- removed link HEBI/elbow/INPUT_INTERFACE
- removed link HEBI/shoulder/INPUT_INTERFACE
- removed link HEBI/wrist/INPUT_INTERFACE
- removed link elbow_wrist1/INPUT_INTERFACE
- removed link shoulder_bracket/INPUT_INTERFACE
- removed link shoulder_elbow/INPUT_INTERFACE
- removed link wrist_paddle/INPUT_INTERFACE
- link base: geometry collision box size=0.25 0.5 0.135; visual box size=0.05 0.05 0.135
- link end_effector/INPUT_INTERFACE: mass None -> 0.0; geometry collision box size=0.01 0.01 0.01; visual box size=0.01 0.01 0.01
Joints:
- removed joint HEBI/base/X5_4
- removed joint HEBI/elbow/X5_4
- removed joint HEBI/shoulder/X5_9
- removed joint HEBI/wrist/X5_9
- removed joint elbow_wrist1/OUTPUT_JOINT
- removed joint shoulder_bracket/OUTPUT_INTERFACE
- removed joint shoulder_elbow/OUTPUT_JOINT
- removed joint wrist_paddle/OUTPUT_JOINT
- joint base_base: child HEBI/base/INPUT_INTERFACE -> end_effector/INPUT_INTERFACE
- joint world_joint: origin xyz=0 0 0 rpy=0 0 0 -> xyz=0 0 -1 rpy=0 0 0

File: hebiros_description/urdf/myArm.xacro (robot description, xacro)
@@ -7,5 +7,5 @@
   <link name="world" />
   <joint name="world_joint"  type="fixed">
-    <origin xyz="0 0 0" rpy="0 0 0" />
+    <origin xyz="0 0 -1" rpy="0 0 0" />
     <parent link="world"/>
     <child link="base"/>
@@ -17,5 +17,5 @@
       <origin xyz="0 0 ${base_height/2}" rpy="0 0 0" />
       <geometry>
-        <box size="0.25 0.5 ${base_height}" />
+        <box size="0.05 0.05 ${base_height}" />
       </geometry>
       <xacro:silver_material/>
@@ -35,9 +35,9 @@
   <joint name="base_base" type="fixed">
     <parent link="base"/>
-    <child link="HEBI/base/INPUT_INTERFACE"/>
+    <child link="end_effector/INPUT_INTERFACE"/>
     <origin xyz="0 0 ${base_height}" rpy="0 0 0"/>
   </joint>
   <!-- joints -->
-  <xacro:x5 joint="HEBI/base" child="shoulder_bracket" model="X5_4"/>
+  <!--<xacro:x5 joint="HEBI/base" child="shoulder_bracket" model="X5_4"/>
   <xacro:x5_heavy_right_outside_bracket name="shoulder_bracket" child="HEBI/shoulder"/>
   <xacro:x5 joint="HEBI/shoulder" child="shoulder_elbow" model="X5_9"/>
@@ -46,7 +46,25 @@
   <xacro:x_tube_link name="elbow_wrist1" child="HEBI/wrist" extension="0.325" twist="${0}"/>
   <xacro:x5 joint="HEBI/wrist" child="wrist_paddle" model="X5_9"/>
-  <xacro:paddle_end name="wrist_paddle" child="end_effector" extension="0.1" paddle_mass=".04" paddle_diameter=".1016"/>
+  <xacro:paddle_end name="wrist_paddle" child="end_effector/INPUT_INTERFACE" extension="0.1" paddle_mass=".04" paddle_diameter=".1016"/>-->
   <!-- end link -->
   <link name="end_effector/INPUT_INTERFACE">
+    <visual>
+      <origin xyz="0 0 0" rpy="0 0 0" />
+      <geometry>
+        <box size="0.01 0.01 0.01" />
+      </geometry>
+      <xacro:silver_material/>
+    </visual>
+    <collision>
+      <origin xyz="0 0 0" rpy="0 0 0" />
+      <geometry>
+        <box size="0.01 0.01 0.01" />
+      </geometry>
+    </collision>
+    <inertial>
+      <origin xyz=".125 0 -.0254" rpy="0 0 0" />
+      <mass value="0.0"/>
+      <inertia ixx="1.0" ixy="0.0" ixz="0.0" iyy="1.0" iyz="0.0" izz="1.0"/>
+    </inertial>
   </link>
   <gazebo reference="base">

Commit message: moved some stuff into my ros folder

File: hebiros_description/urdf/myArm.urdf (robot description, URDF)
Before this commit: robot CNU_HEBI_Arm, 3 links, 2 joints
Links:
- added link HEBI/base/INPUT_INTERFACE, mass 0.335; collision mesh filename=package://hebiros_description/meshes/x5.stl scale=0.001 0.001 0.001; visual mesh filename=package://hebiros_description/meshes/x5.stl scale=0.001 0.001 0.001
- added link HEBI/elbow/INPUT_INTERFACE, mass 0.335; collision mesh filename=package://hebiros_description/meshes/x5.stl scale=0.001 0.001 0.001; visual mesh filename=package://hebiros_description/meshes/x5.stl scale=0.001 0.001 0.001
- added link HEBI/shoulder/INPUT_INTERFACE, mass 0.360; collision mesh filename=package://hebiros_description/meshes/x5.stl scale=0.001 0.001 0.001; visual mesh filename=package://hebiros_description/meshes/x5.stl scale=0.001 0.001 0.001
- added link HEBI/wrist/INPUT_INTERFACE, mass 0.360; collision mesh filename=package://hebiros_description/meshes/x5.stl scale=0.001 0.001 0.001; visual mesh filename=package://hebiros_description/meshes/x5.stl scale=0.001 0.001 0.001
- added link elbow_wrist1/INPUT_INTERFACE, mass 0.402; collision cylinder length=0.2996 radius=.016; collision mesh filename=package://hebiros_description/meshes/A-2038-02.stl
- added link shoulder_bracket/INPUT_INTERFACE, mass 0.215; collision mesh filename=package://hebiros_description/meshes/PM-2149-01.stl scale=0.001 0.001 0.001; collision mesh filename=package://hebiros_description/meshes/PM-2150-01R.stl scale=0.001 0.001 0.001
- added link shoulder_elbow/INPUT_INTERFACE, mass 0.402; collision cylinder length=0.2996 radius=.016; collision mesh filename=package://hebiros_description/meshes/A-2038-02.stl
- added link wrist_paddle/INPUT_INTERFACE, mass 0.312; collision cylinder length=0.025 radius=0.0508; collision cylinder length=0.075 radius=.016
Joints:
- added joint HEBI/base/X5_4: type continuous, parent HEBI/base/INPUT_INTERFACE, child shoulder_bracket/INPUT_INTERFACE, origin xyz=0 0 0.031 rpy=0 0 0, axis 0 0 1, limit effort=7.0 velocity=32
- added joint HEBI/elbow/X5_4: type continuous, parent HEBI/elbow/INPUT_INTERFACE, child elbow_wrist1/INPUT_INTERFACE, origin xyz=0 0 0.031 rpy=0 0 0, axis 0 0 1, limit effort=7.0 velocity=32
- added joint HEBI/shoulder/X5_9: type continuous, parent HEBI/shoulder/INPUT_INTERFACE, child shoulder_elbow/INPUT_INTERFACE, origin xyz=0 0 0.031 rpy=0 0 0, axis 0 0 1, limit effort=13.0 velocity=14
- added joint HEBI/wrist/X5_9: type continuous, parent HEBI/wrist/INPUT_INTERFACE, child wrist_paddle/INPUT_INTERFACE, origin xyz=0 0 0.031 rpy=0 0 0, axis 0 0 1, limit effort=13.0 velocity=14
- added joint elbow_wrist1/OUTPUT_JOINT: type fixed, parent elbow_wrist1/INPUT_INTERFACE, child HEBI/wrist/INPUT_INTERFACE, origin xyz=0.325 -0.0 0.04 rpy=0 0 0
- added joint shoulder_bracket/OUTPUT_INTERFACE: type fixed, parent shoulder_bracket/INPUT_INTERFACE, child HEBI/shoulder/INPUT_INTERFACE, origin xyz=0 -.0375 .055 rpy=1.57079632679 0 0
- added joint shoulder_elbow/OUTPUT_JOINT: type fixed, parent shoulder_elbow/INPUT_INTERFACE, child HEBI/elbow/INPUT_INTERFACE, origin xyz=0.325 -0.02 0.02 rpy=1.57079632679 0 0
- added joint wrist_paddle/OUTPUT_JOINT: type fixed, parent wrist_paddle/INPUT_INTERFACE, child end_effector/INPUT_INTERFACE, origin xyz=0 0 0.1 rpy=0 0 0
- joint base_base: child end_effector/INPUT_INTERFACE -> HEBI/base/INPUT_INTERFACE
- joint world_joint: origin xyz=0 0 -1 rpy=0 0 0 -> xyz=0 0 0 rpy=0 0 0

File: hebiros_description/urdf/myArm.xacro (robot description, xacro)
@@ -6,5 +6,5 @@
   <!-- ************************* ROBOT DEFINITION ************************* -->
   <link name="world" />
-  <joint name="world_joint"  type="fixed">guages, like human bodies, come in a variety of shapes—but only to a point. Just as people don’t sprout multiple heads, languages tend to veer away from certain forms that might spring from an imaginative mind. For example, one core property of human languages is known as duality of patterning: meaningful linguistic units (such as words) break down into smaller meaningless units (sounds), so that the words sap, pass, and asp inv
+  <joint name="world_joint"  type="fixed">
     <origin xyz="0 0 0" rpy="0 0 0" />
     <parent link="world"/>
