Commit message: ugh

File: hebiros_description/urdf/x_demo.xacro (robot description, xacro)
@@ -36,7 +36,7 @@
     <origin xyz="0 0 0" rpy="0 0 0"/>
   </joint>
-  <!-- joints -->
+  <!-- joints-->
   <xacro:x5 joint="HEBI/base" child="shoulder_bracket" model="X5_4"/>
-  <xacro:x5_heavy_right_inside_bracket name="shoulder_bracket" child="HEBI/shoulder"/>
+  <xacro:x5_heavy_right_outside_bracket name="shoulder_bracket" child="HEBI/shoulder"/>
   <xacro:x5 joint="HEBI/shoulder" child="shoulder_elbow" model="X5_4"/>
   <xacro:x_tube_link name="shoulder_elbow" child="HEBI/elbow" extension="0.33" twist="${PI}"/>
@@ -45,4 +45,22 @@
   <!-- end link -->
   <link name="end_effector/INPUT_INTERFACE">
+    <visual>
+      <origin xyz="0 0 0" rpy="0 0 0" />
+      <geometry>
+        <box size="0.01 0.01 0.01" />
+      </geometry>
+      <xacro:silver_material/>
+    </visual>
+    <collision>
+      <origin xyz="0 0 0" rpy="0 0 0" />
+      <geometry>
+        <box size="0.01 0.01 0.01" />
+      </geometry>
+    </collision>
+    <inertial>
+      <origin xyz=".125 0 -.0254" rpy="0 0 0" />
+      <mass value="0.0"/>
+      <inertia ixx="1.0" ixy="0.0" ixz="0.0" iyy="1.0" iyz="0.0" izz="1.0"/>
+    </inertial>
   </link>
   <gazebo reference="base">
