Commit message: start for day

File: hebiros_description/urdf/myArm.xacro (robot description, xacro)
@@ -1,12 +1,7 @@
 <?xml version="1.0"?>
-<robot name="arm_demo">
+<!-- HEBI 6-DOF Robot arm kit -->
+<robot xmlns:xacro="http://www.ros.org/wiki/xacro" name="A-2085-06">
   <!-- *************************** XACRO MACROS *************************** -->
-  <xacro:property name="PI" value="3.1415926535897931" />
-  <!-- load macros for modules -->
-  <xacro:include filename="./x_series_common.xacro"/>
-  <xacro:include filename="./x5.xacro"/>
-  <xacro:include filename="./x_shoulder_bracket.xacro"/>
-  <xacro:include filename="./x_wrist_bracket.xacro"/>
-  <xacro:include filename="./x_tube_link.xacro"/>
+  <xacro:include filename="./x_library.xacro"/>
   <!-- ************************* ROBOT DEFINITION ************************* -->
   <link name="world" />
@@ -19,5 +14,5 @@
   <link name="base">
     <visual>
-      <origin xyz=".125 0 -.0254" rpy="0 0 0" />
+      <origin xyz="-.125 0 -.0254" rpy="0 0 0" />
       <geometry>
         <box size="0.25 0.5 0.0508" />
@@ -26,5 +21,5 @@
     </visual>
     <collision>
-      <origin xyz=".125 0 -.0254" rpy="0 0 0" />
+      <origin xyz="-.125 0 -.0254" rpy="0 0 0" />
       <geometry>
         <box size="0.25 0.5 0.0508" />
@@ -43,6 +38,11 @@
   </joint>
   <!-- joints -->
-  <xacro:x5 joint="HEBI/base" child="base_end" model="X5-4"/>
-  <xacro:x_tube_link name="base_end" child="end_effector" length="0.33" twist="0"/>
+  <xacro:x5 joint="HEBI/base" child="shoulder_bracket" model="X5_4"/>
+  <xacro:x5_heavy_right_outside_bracket name="shoulder_bracket" child="HEBI/shoulder"/>
+  <xacro:x5 joint="HEBI/shoulder" child="shoulder_elbow" model="X5_9"/>
+  <xacro:x_tube_link name="shoulder_elbow" child="HEBI/elbow" extension="0.325" twist="${PI/2}"/>
+  <xacro:x5 joint="HEBI/elbow" child="elbow_wrist1" model="X5_4"/>
+  <xacro:x_tube_link name="elbow_wrist1" child="HEBI/wrist1" extension="0.325" twist="${0}"/>
+  <xacro:x5 joint="HEBI/wrist1" child="end_effector" model="X5_9"/>
   <!-- end link -->
   <link name="end_effector/INPUT_INTERFACE">

Commit message: arm looks good

File: hebiros_description/urdf/myArm.xacro (robot description, xacro)
@@ -12,16 +12,17 @@
   </joint>
   <!-- just for visualization: base post -->
+  <xacro:property name="base_height" value="${.135}"/>
   <link name="base">
     <visual>
-      <origin xyz="-.125 0 -.0254" rpy="0 0 0" />
+      <origin xyz="0 0 ${base_height/2}" rpy="0 0 0" />
       <geometry>
-        <box size="0.25 0.5 0.0508" />
+        <box size="0.25 0.5 ${base_height}" />
       </geometry>
       <xacro:silver_material/>
     </visual>
     <collision>
-      <origin xyz="-.125 0 -.0254" rpy="0 0 0" />
+      <origin xyz="0 0 ${base_height/2}" rpy="0 0 0" />
       <geometry>
-        <box size="0.25 0.5 0.0508" />
+        <box size="0.25 0.5 ${base_height}" />
       </geometry>
     </collision>
@@ -35,5 +36,5 @@
     <parent link="base"/>
     <child link="HEBI/base/INPUT_INTERFACE"/>
-    <origin xyz="0 0 0" rpy="0 0 0"/>
+    <origin xyz="0 0 ${base_height}" rpy="0 0 0"/>
   </joint>
   <!-- joints -->
@@ -45,5 +46,5 @@
   <xacro:x_tube_link name="elbow_wrist1" child="HEBI/wrist" extension="0.325" twist="${0}"/>
   <xacro:x5 joint="HEBI/wrist" child="wrist_paddle" model="X5_9"/>
-  <xacro:paddle_end name="wrist_paddle" child="end_effector" extension="0.1"/>
+  <xacro:paddle_end name="wrist_paddle" child="end_effector" extension="0.1" paddle_mass=".04" paddle_diameter=".1016"/>
   <!-- end link -->
   <link name="end_effector/INPUT_INTERFACE">

File: hebiros_description/urdf/paddle_end.xacro (robot description, xacro)
@@ -2,25 +2,49 @@
 <robot xmlns:xacro="http://www.ros.org/wiki/xacro">
   <!-- NOTE: joint must match the name of the module -->
-  <xacro:macro name="paddle_end" params="name child extension">
-    <xacro:property name="mass" value="${0.4 * (extension + 0.03) + 0.26}"/>
+  <xacro:macro name="paddle_end" params="name child extension paddle_mass paddle_diameter">
+    <xacro:property name="tube_mass" value="${0.4 * (extension + 0.03) + 0.26}"/>
+    <xacro:property name="edge_to_center" value="${.02}"/>
+    <xacro:property name="paddle_height" value="${.025}"/>
     <link name="${name}/INPUT_INTERFACE">
       <visual>
-        <origin xyz="${extension/2} 0 0" rpy="0 0 0" />
+        <origin xyz="0 0 ${(extension-paddle_height)/2}" rpy="0 0 0" />
         <geometry>
-          <cylinder length="${extension-.0254}" radius=".016" />
+          <cylinder length="${extension-paddle_height}" radius=".016" />
         </geometry>
-        <xacro:silver_material/>
+        <material name="orange">
+          <color rgba="${255/255} ${108/255} ${10/255} 1.0"/>
+        </material>
+      </visual>
+      <visual>
+        <origin xyz="0 0 ${extension-(paddle_height/2)}" rpy="0 0 0" />
+        <geometry>
+          <cylinder length="${paddle_height}" radius="${paddle_diameter/2}"/>
+        </geometry>
+        <material name="orange">
+          <color rgba="${255/255} ${108/255} ${10/255} 1.0"/>
+        </material>
       </visual>
       <collision>
-        <origin xyz="${extension/2} 0 0" rpy="0 0 0"/>
+        <origin xyz="0 0 ${(extension-paddle_height)/2}" rpy="0 0 0" />
         <geometry>
-          <cylinder length="${extension-.0254}" radius=".016" />
+          <cylinder length="${extension-paddle_height}" radius=".016" />
+        </geometry>
+      </collision>
+      <collision>
+        <origin xyz="0 0 ${extension-(paddle_height/2)}" rpy="0 0 0" />
+        <geometry>
+          <cylinder length="${paddle_height}" radius="${paddle_diameter/2}" />
         </geometry>
       </collision>
       <!-- Approximate inertia as thin rod about x axis -->
       <inertial>
-        <origin xyz="${extension/2} 0 0" rpy="0 0 0" />
-        <mass value="${mass}"/>
-        <inertia  ixx="0.0" ixy="0.0"  ixz="0.0"  iyy="${mass * extension * extension / 12.0}"  iyz="0.0"  izz="${mass * extension * extension / 12.0}"/>
+        <origin xyz="0 0 ${(extension-paddle_height)/2}" rpy="0 0 0" />
+        <mass value="${tube_mass}"/>
+        <inertia  ixx="0.0" ixy="0.0"  ixz="0.0"  iyy="${tube_mass * extension * extension / 12.0}"  iyz="0.0"  izz="${tube_mass * extension * extension / 12.0}"/>
+      </inertial>
+      <inertial>
+        <origin xyz="0 0 ${extension-(paddle_height/2)}" rpy="0 0 0" />
+        <mass value="${paddle_mass}"/>
+        <inertia  ixx="0.0" ixy="0.0"  ixz="0.0"  iyy="${paddle_mass * paddle_height * paddle_height / 12.0}"  iyz="0.0"  izz="${paddle_mass * paddle_height * paddle_height / 12.0}"/>
       </inertial>
     </link>
@@ -28,5 +52,5 @@
       <parent link="${name}/INPUT_INTERFACE"/>
       <child link="${child}/INPUT_INTERFACE"/>
-      <origin xyz="${extension} 0 0" rpy="0 0 0"/>
+      <origin xyz="0 0 ${extension}" rpy="0 0 0"/>
     </joint>
     <gazebo reference="${name}/INPUT_INTERFACE">

File: hebiros_description/urdf/x_library.xacro (robot description, xacro)
@@ -12,3 +12,4 @@
   <xacro:include filename="./x5_heavy_right_inside_bracket.xacro"/>
   <xacro:include filename="./x_tube_link.xacro"/>
+  <xacro:include filename="./paddle_end.xacro"/>
 </robot>

Commit message: nothing as it should be

File: hebiros_description/urdf/myArm.xacro (robot description, xacro)
@@ -7,5 +7,5 @@
   <link name="world" />
   <joint name="world_joint"  type="fixed">
-    <origin xyz="0 0 -1" rpy="0 0 0" />
+    <origin xyz="0 0 0" rpy="0 0 0" />
     <parent link="world"/>
     <child link="base"/>
@@ -35,9 +35,9 @@
   <joint name="base_base" type="fixed">
     <parent link="base"/>
-    <child link="end_effector/INPUT_INTERFACE"/>
+    <child link="HEBI/base/INPUT_INTERFACE"/>
     <origin xyz="0 0 ${base_height}" rpy="0 0 0"/>
   </joint>
   <!-- joints -->
-  <!--<xacro:x5 joint="HEBI/base" child="shoulder_bracket" model="X5_4"/>
+  <xacro:x5 joint="HEBI/base" child="shoulder_bracket" model="X5_4"/>
   <xacro:x5_heavy_right_outside_bracket name="shoulder_bracket" child="HEBI/shoulder"/>
   <xacro:x5 joint="HEBI/shoulder" child="shoulder_elbow" model="X5_9"/>
@@ -46,5 +46,5 @@
   <xacro:x_tube_link name="elbow_wrist1" child="HEBI/wrist" extension="0.325" twist="${0}"/>
   <xacro:x5 joint="HEBI/wrist" child="wrist_paddle" model="X5_9"/>
-  <xacro:paddle_end name="wrist_paddle" child="end_effector/INPUT_INTERFACE" extension="0.1" paddle_mass=".04" paddle_diameter=".1016"/>-->
+  <xacro:paddle_end name="wrist_paddle" child="end_effector" extension="0.1" paddle_mass=".04" paddle_diameter=".1016"/>
   <!-- end link -->
   <link name="end_effector/INPUT_INTERFACE">

Commit message: my arm xacro changes

File: hebiros_description/urdf/myArm.xacro (robot description, xacro)
@@ -6,5 +6,5 @@
   <!-- ************************* ROBOT DEFINITION ************************* -->
   <link name="world" />
-  <joint name="world_joint"  type="fixed">
+  <joint name="world_joint"  type="fixed">guages, like human bodies, come in a variety of shapes—but only to a point. Just as people don’t sprout multiple heads, languages tend to veer away from certain forms that might spring from an imaginative mind. For example, one core property of human languages is known as duality of patterning: meaningful linguistic units (such as words) break down into smaller meaningless units (sounds), so that the words sap, pass, and asp inv
     <origin xyz="0 0 0" rpy="0 0 0" />
     <parent link="world"/>

Commit message: added a trajectory single control for my arm

File: hebiros_description/urdf/myArm.xacro (robot description, xacro)
@@ -24,5 +24,5 @@
       <origin xyz="0 0 ${base_height/2}" rpy="0 0 0" />
       <geometry>
-        <box size="0.25 0.5 ${base_height}" />
+        <box size="0.05 0.5 ${base_height}" />
       </geometry>
     </collision>
